Commit message: Adapted to Kate Changed connection joint

File: kurt_description/tops/kurtana_top.urdf.xacro (robot description, xacro)
@@ -10,6 +10,7 @@
   <!-- ******************** -->
   <include filename="$(find kurt_description)/parts/kurtana_rack.urdf.xacro" />
-  <property name="kinect_x_offset" value="0.018" />
-  <property name="kinect_z_offset" value="0.087" />
+  <property name="kinect_x_offset" value="0.03" />
+  <property name="kinect_y_offset" value="0.0" />
+  <property name="kinect_z_offset" value="0.018" />
   <!-- ************************ -->
   <!-- *** Microsoft Kinect *** -->
@@ -18,7 +19,7 @@
   <xacro:kinect camera="kinect" />
   <joint name="kurtana_kinect_joint" type="fixed">
-    <parent link="kurtana_pitchpole_link" />
+    <parent link="kurtana_kinect_mounting_plate_link" />
     <child  link="kinect_link" />
-    <origin xyz="${kinect_x_offset} 0 ${kinect_z_offset}" rpy="0 0 0"/>
+    <origin xyz="${kinect_x_offset} ${kinect_y_offset} ${kinect_z_offset}" rpy="0 0 0"/>
   </joint>
   <!-- ************************* -->
@@ -35,15 +36,11 @@
   <!-- *** Neuronics Katana Arm *** -->
   <!-- **************************** -->
-  <include filename="$(find katana_description)/urdf/katana_450_6m90a_with_controlbox.urdf.xacro" />
-  <link name="katana_pattern"></link>
-  <joint name="katana_pattern_joint" type="fixed">
-    <parent link="katana_motor4_lift_link"/>
-    <child  link="katana_pattern" />
-    <origin xyz=".075 -.035 0.00" rpy="1.571 -1.571 0.151"/>
-  </joint>
-  <joint name="kurtana_baseplate_controlbox_joint" type="fixed">
-    <parent link="kurtana_baseplate_link" />
-    <child link="katana_internal_controlbox_link" />
-    <origin xyz="0.05 0 ${baseplate_height*1.5}" rpy="0 0 0" />
+ <include filename="$(find katana_description)/urdf/katana_300_6m180.urdf.xacro" />
+ <!-- send katana urdf to param server
+  <param name="robot_description" command="$(find xacro)/xacro.py '$(find katana_description)/urdf/katana_300_6m180.urdf.xacro'" /> -->
+  <joint name="kurtana_baseplate_katana_baseplate_joint" type="fixed">
+    <parent link="katana_baseplate_link" />
+    <child link="katana_base_link" />
+    <origin xyz="0 0 0" rpy="0 0 0" />
   </joint>
 </robot>

Commit message: Removed Kinect offsets (not suitable for the ptu) Adde Kinect calibration pattern link

File: kurt_description/tops/kurtana_top.urdf.xacro (robot description, xacro)
@@ -10,7 +10,8 @@
   <!-- ******************** -->
   <include filename="$(find kurt_description)/parts/kurtana_rack.urdf.xacro" />
-  <property name="kinect_x_offset" value="0.03" />
+ <!-- these offsets shouldn't be used if the Kinect is on a PTU-->
+  <property name="kinect_x_offset" value="0.0" />
   <property name="kinect_y_offset" value="0.0" />
-  <property name="kinect_z_offset" value="0.018" />
+  <property name="kinect_z_offset" value="0.0" />
   <!-- ************************ -->
   <!-- *** Microsoft Kinect *** -->
@@ -22,14 +23,4 @@
     <child  link="kinect_link" />
     <origin xyz="${kinect_x_offset} ${kinect_y_offset} ${kinect_z_offset}" rpy="0 0 0"/>
-  </joint>
-  <!-- ************************* -->
-  <!-- *** SICK TiM3xx laser *** -->
-  <!-- ************************* -->
-  <include filename="$(find sick_tim3xx)/urdf/sick_tim3xx.urdf.xacro" />
-  <xacro:sick_tim3xx laser_link="laser" />
-  <joint name="kurtana_laser_joint" type="fixed">
-    <parent link="kurtana_baseplate_link" />
-    <child link="laser_mount_link" />
-    <origin xyz="${baseplate_length/2 - sick_tim3xx_length/2} 0 ${baseplate_height/2}" rpy="0 0 0" />
   </joint>
   <!-- **************************** -->
@@ -44,3 +35,10 @@
     <origin xyz="0 0 0" rpy="0 0 0" />
   </joint>
+  <!-- pattern for Kinect calibration -->
+   <link name="katana_pattern"></link>
+  <joint name="katana_pattern_joint" type="fixed">
+    <parent link="katana_motor4_lift_link"/>
+    <child  link="katana_pattern" />
+    <origin xyz=".075 -.035 0.00" rpy="1.571 -1.571 0.151"/>
+  </joint>
 </robot>
